File: ads1115with16JTS.kicad_sch (KiCad schematic)
At the start: 41 parts, among them J1 Conn_01x02_Pin, J10 Conn_01x02_Pin, J11 Conn_01x02_Pin, J12 Conn_01x02_Pin, J13 Conn_01x02_Pin, J14 Conn_01x02_Pin, J15 Conn_01x02_Pin, J16 Conn_01x02_Pin, J17 Conn_01x04_Pin, J2 Conn_01x02_Pin, J3 Conn_01x02_Pin, J4 Conn_01x02_Pin, J5 Conn_01x02_Pin, J6 Conn_01x02_Pin, J7 Conn_01x02_Pin, J8 Conn_01x02_Pin, J9 Conn_01x02_Pin, U1 ADS1115IDGS, U2 ADS1115IDGS, U3 ADS1115IDGS, U4 ADS1115IDGS

Commit message: snapshot v0.0.10
Parts:
- added J18: PinSocket_1x20_P2.54mm_Vertical, PG:b_pill_socket_1-20, symbol PG:b_pill_1-20
- added J19: PinSocket_1x20_P2.54mm_Vertical, PG:b_pill_socket_21-40, symbol PG:b_pill_21-40
- added pads1: SolderWire-0.25sqmm_1x04_P4.2mm_D0.65mm_OD1.7mm, SolderWire-0.25sqmm_1x04_P4.2mm_D0.65mm_OD1.7mm, symbol Connector:Conn_01x04_Pin
- added pads2: SolderWire-0.25sqmm_1x20_P4.2mm_D0.65mm_OD1.7mm, PG:b_pill_socket_1-20, symbol PG:b_pill_1-20
- added pads3: SolderWire-0.25sqmm_1x20_P4.2mm_D0.65mm_OD1.7mm, PG:b_pill_takeoffPads_21-40, symbol PG:b_pill_21-40
- J1, J10, J11, J12, J13, J14, J15, J16, J2, J3, J4, J5, J6, J7, J8, J9: footprint Connector_JST:JST_XH_S2B-XH-A_1x02_P2.50mm_Horizontal -> Connector_JST:JST_XH_B2B-XH-A_1x02_P2.50mm_Vertical
- R1, R10, R11, R12, R13, R14, R15, R16, R2, R3, R4, R5, R6, R7, R8, R9: footprint Resistor_SMD:R_0805_2012Metric -> Resistor_SMD:R_0603_1608Metric
Connections:
- net +3V3: now also J19.40 (3v3), pads1.2 (Pin_2), pads3.40 (3v3)
- net GND: now also J19.39 (G), pads1.1 (Pin_1), pads3.39 (G)
- net SCL1: now reaches J17.4 (Pin_4), U1.10 (SCL), U2.10 (SCL), U3.10 (SCL), U4.1 (ADDR), U4.10 (SCL)
- net SCL1: now also J19.36 (B8), pads1.4 (Pin_4), pads3.36 (B8)
- net SDA1: now reaches J17.3 (Pin_3), U1.9 (SDA), U2.9 (SDA), U3.1 (ADDR), U3.9 (SDA), U4.9 (SDA)
- net SDA1: now also J19.37 (B9), pads1.3 (Pin_3), pads3.37 (B9)
- new net: J19.21, pads3.21
- new net: J19.22, pads3.22
- new net: J19.23, pads3.23
- new net: J19.24, pads3.24
- new net: J19.25, pads3.25
- new net: J19.26, pads3.26
- new net: J19.27, pads3.27
- new net: J19.28, pads3.28
- new net: J19.29, pads3.29
- new net: J19.30, pads3.30
- new net: J19.32, pads3.32
- new net: J19.33, pads3.33
- new net: J19.34, pads3.34
- new net: J19.35, pads3.35
- new net: J19.38 (5v), pads3.38 (5v)
- new net: J18.1, pads2.1
- new net: J18.10, pads2.10
- new net: J18.11, pads2.11
- new net: J18.12, pads2.12
- new net: J18.13, pads2.13
- new net: J18.14, pads2.14
- new net: J18.15, pads2.15
- new net: J18.16, pads2.16
- new net: J18.18 (3v3), pads2.18 (3v3)
- new net: J18.19 (G), pads2.19 (G)
- new net: J18.2, pads2.2
- new net: J18.20 (5v), pads2.20 (5v)
- new net: J18.3, pads2.3
- new net: J18.4, pads2.4
- new net: J18.5, pads2.5
- new net: J18.6, pads2.6
- new net: J18.7, pads2.7
- new net: J18.8, pads2.8
- new net: J18.9, pads2.9
- new net SCL2: J18.17 (B10), pads2.17 (B10)
- new net SDA2: J19.31 (B3), pads3.31 (B3)
Other:
- moved on the sheet: J17

Commit message: changes for v0.0.12
Parts:
- J**1: renamed from pads2; footprint PG:b_pill_socket_1-20 -> PG:b_pill_takeoffPads_1-20; symbol PG:b_pill_1-20 -> PG:b_pill_takeoff_1-20
- J**2: renamed from pads3; value SolderWire-0.25sqmm_1x20_P4.2mm_D0.65mm_OD1.7mm -> SolderWire-0.25sqmm_1x20_P4.2mm_D0.65mm_OD1.7mm; symbol PG:b_pill_21-40 -> PG:b_pill_takeoff_21-40
Other:
- moved on the sheet: J18
Changed lines of the file:
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@@
   (junction (at 78.74 88.9) (diameter 0) (color 0 0 0 0)
   )
+  (junction (at 184.15 102.87) (diameter 0) (color 0 0 0 0)
+  )
+  (junction (at 140.97 166.37) (diameter 0) (color 0 0 0 0)
+  )
+  (junction (at 128.27 196.85) (diameter 0) (color 0 0 0 0)
+  )
+  (junction (at 48.26 66.04) (diameter 0) (color 0 0 0 0)
+  )
+  (junction (at 140.97 67.31) (diameter 0) (color 0 0 0 0)
+  )
+  (junction (at 125.73 171.45) (diameter 0) (color 0 0 0 0)
+  )
+  (junction (at 184.15 53.34) (diameter 0) (color 0 0 0 0)
+  )
+  (junction (at 125.73 142.24) (diameter 0) (color 0 0 0 0)
+  )
   (junction (at 143.51 104.14) (diameter 0) (color 0 0 0 0)
-  )
-  (junction (at 184.15 102.87) (diameter 0) (color 0 0 0 0)
-  )
-  (junction (at 140.97 166.37) (diameter 0) (color 0 0 0 0)
-  )
-  (junction (at 128.27 196.85) (diameter 0) (color 0 0 0 0)
-  )
-  (junction (at 48.26 66.04) (diameter 0) (color 0 0 0 0)
-  )
-  (junction (at 140.97 67.31) (diameter 0) (color 0 0 0 0)
-  )
-  (junction (at 125.73 171.45) (diameter 0) (color 0 0 0 0)
-  )
-  (junction (at 184.15 53.34) (diameter 0) (color 0 0 0 0)
-  )
-  (junction (at 125.73 142.24) (diameter 0) (color 0 0 0 0)
   )
   (junction (at 184.15 64.77) (diameter 0) (color 0 0 0 0)
@@
   (no_connect (at 138.43 210.82))
   (no_connect (at 135.89 99.06))
-  (wire (pts (xy 152.4 148.59) (xy 157.48 148.59))
+  (wire (pts (xy 157.48 148.59) (xy 162.56 148.59))
     (stroke (width 0) (type default))
   )
@@
     (stroke (width 0) (type default))
   )
-  (wire (pts (xy 152.4 130.81) (xy 157.48 130.81))
+  (wire (pts (xy 157.48 130.81) (xy 162.56 130.81))
     (stroke (width 0) (type default))
   )
@@
     (stroke (width 0) (type default))
   )
-  (wire (pts (xy 152.4 138.43) (xy 157.48 138.43))
+  (wire (pts (xy 157.48 138.43) (xy 162.56 138.43))
     (stroke (width 0) (type default))
   )
@@
     (stroke (width 0) (type default))
   )
-  (wire (pts (xy 152.4 128.27) (xy 157.48 128.27))
+  (wire (pts (xy 157.48 128.27) (xy 162.56 128.27))
     (stroke (width 0) (type default))
   )
@@
     (stroke (width 0) (type default))
   )
-  (wire (pts (xy 152.4 133.35) (xy 157.48 133.35))
-    (stroke (width 0) (type default))
-  )
-  (wire (pts (xy 152.4 146.05) (xy 157.48 146.05))
+  (wire (pts (xy 157.48 133.35) (xy 162.56 133.35))
+    (stroke (width 0) (type default))
+  )
+  (wire (pts (xy 157.48 146.05) (xy 162.56 146.05))
     (stroke (width 0) (type default))
   )
@@
     (stroke (width 0) (type default))
   )
-  (wire (pts (xy 152.4 123.19) (xy 157.48 123.19))
+  (wire (pts (xy 157.48 123.19) (xy 162.56 123.19))
     (stroke (width 0) (type default))
   )
@@
     (stroke (width 0) (type default))
   )
-  (wire (pts (xy 152.4 143.51) (xy 157.48 143.51))
+  (wire (pts (xy 133.35 123.19) (xy 138.43 123.19))
+    (stroke (width 0) (type default))
+  )
+  (wire (pts (xy 157.48 143.51) (xy 162.56 143.51))
     (stroke (width 0) (type default))
   )
@@
     (stroke (width 0) (type default))
   )
-  (wire (pts (xy 152.4 102.87) (xy 157.48 102.87))
+  (wire (pts (xy 157.48 102.87) (xy 162.56 102.87))
     (stroke (width 0) (type default))
   )
@@
     (stroke (width 0) (type default))
   )
-  (wire (pts (xy 152.4 107.95) (xy 157.48 107.95))
+  (wire (pts (xy 157.48 107.95) (xy 162.56 107.95))
     (stroke (width 0) (type default))
   )
@@
     (stroke (width 0) (type default))
   )
-  (wire (pts (xy 152.4 118.11) (xy 157.48 118.11))
+  (wire (pts (xy 157.48 118.11) (xy 162.56 118.11))
     (stroke (width 0) (type default))
   )
@@
     (stroke (width 0) (type default))
   )
-  (wire (pts (xy 152.4 110.49) (xy 157.48 110.49))
+  (wire (pts (xy 157.48 110.49) (xy 162.56 110.49))
     (stroke (width 0) (type default))
   )
@@
     (stroke (width 0) (type default))
   )
-  (wire (pts (xy 152.4 140.97) (xy 157.48 140.97))
+  (wire (pts (xy 157.48 140.97) (xy 162.56 140.97))
     (stroke (width 0) (type default))
   )
@@
     (stroke (width 0) (type default))
   )
-  (wire (pts (xy 152.4 105.41) (xy 157.48 105.41))
+  (wire (pts (xy 157.48 105.41) (xy 162.56 105.41))
     (stroke (width 0) (type default))
   )
@@
     (stroke (width 0) (type default))
   )
-  (wire (pts (xy 152.4 120.65) (xy 157.48 120.65))
+  (wire (pts (xy 157.48 120.65) (xy 162.56 120.65))
     (stroke (width 0) (type default))
   )
@@
     (stroke (width 0) (type default))
   )
-  (wire (pts (xy 152.4 135.89) (xy 157.48 135.89))
+  (wire (pts (xy 157.48 135.89) (xy 162.56 135.89))
     (stroke (width 0) (type default))
   )
@@
     (stroke (width 0) (type default))
   )
-  (wire (pts (xy 152.4 151.13) (xy 157.48 151.13))
+  (wire (pts (xy 157.48 151.13) (xy 162.56 151.13))
     (stroke (width 0) (type default))
   )
@@
     (stroke (width 0) (type default))
   )
-  (wire (pts (xy 133.35 123.19) (xy 138.43 123.19))
-    (stroke (width 0) (type default))
-  )
   (wire (pts (xy 81.28 227.33) (xy 88.9 227.33))
     (stroke (width 0) (type default))
@@
     (stroke (width 0) (type default))
   )
-  (wire (pts (xy 152.4 115.57) (xy 157.48 115.57))
+  (wire (pts (xy 157.48 115.57) (xy 162.56 115.57))
     (stroke (width 0) (type default))
   )
@@
     (stroke (width 0) (type default))
   )
-  (wire (pts (xy 152.4 125.73) (xy 157.48 125.73))
+  (wire (pts (xy 157.48 125.73) (xy 162.56 125.73))
     (stroke (width 0) (type default))
   )
@@
     (stroke (width 0) (type default))
   )
-  (wire (pts (xy 152.4 113.03) (xy 157.48 113.03))
+  (wire (pts (xy 157.48 113.03) (xy 162.56 113.03))
     (stroke (width 0) (type default))
   )
@@
     (stroke (width 0) (type default))
   )
-  (label "SCL2" (at 152.4 143.51 0) (fields_autoplaced)
+  (label "SCL2" (at 157.48 143.51 0) (fields_autoplaced)
     (effects (font (size 1.27 1.27)) (justify left bottom))
   )
@@
       (effects (font (size 2.54 2.54)))
     )
-    (property "Value" "PinSocket_1x20_P2.54mm_Vertical" (at 199.39 135.89 90)
-      (effects (font (size 1.27 1.27)))
-    )
-    (property "Footprint" "PG:b_pill_socket_21-40" (at 199.39 101.6 90) (show_name)
+    (property "Value" "PinSocket_1x20_P2.54mm_Vertical" (at 199.39 132.08 90)
+      (effects (font (size 1.27 1.27)))
+    )
+    (property "Footprint" "PG:b_pill_socket_21-40" (at 201.93 132.08 90) (show_name)
       (effects (font (size 1.27 1.27)))
     )
@@
     )
   )
-  (symbol (lib_id "PG:b_pill_1-20") (at 137.16 128.27 0) (mirror y) (unit 1)
+  (symbol (lib_id "PG:b_pill_1-20") (at 157.48 128.27 0) (unit 1)
     (in_bom yes) (on_board yes) (dnp no)
     (property "Reference" "J18" (at 151.13 156.21 0)
       (effects (font (size 2.54 2.54)) (justify left))
     )
-    (property "Value" "PinSocket_1x20_P2.54mm_Vertical" (at 144.78 143.51 90)
+    (property "Value" "PinSocket_1x20_P2.54mm_Vertical" (at 149.86 140.97 90)
       (effects (font (size 1.27 1.27)) (justify left))
     )
-    (property "Footprint" "PG:b_pill_socket_1-20" (at 142.24 142.24 90) (show_name)
+    (property "Footprint" "PG:b_pill_socket_1-20" (at 147.32 139.7 90) (show_name)
       (effects (font (size 1.27 1.27)) (justify left))
     )
-    (property "Datasheet" "" (at 137.16 128.27 0)
+    (property "Datasheet" "" (at 142.24 128.27 0)
       (effects (font (size 1.27 1.27)) hide)
     )
@@
     )
   )
-  (symbol (lib_id "PG:b_pill_1-20") (at 172.72 128.27 0) (unit 1)
+  (symbol (lib_id "PG:b_pill_takeoff_1-20") (at 160.02 128.27 0) (mirror y) (unit 1)
     (in_bom yes) (on_board yes) (dnp no)
-    (property "Reference" "pads2" (at 156.21 156.21 0)
-      (effects (font (size 2.54 2.54)) (justify left))
-    )
-    (property "Value" "SolderWire-0.25sqmm_1x20_P4.2mm_D0.65mm_OD1.7mm" (at 165.1 153.67 90)
-      (effects (font (size 1.27 1.27)) (justify left))
-    )
-    (property "Footprint" "PG:b_pill_socket_1-20" (at 167.64 147.32 90) (show_name)
-      (effects (font (size 1.27 1.27)) (justify left))
-    )
-    (property "Datasheet" "" (at 172.72 128.27 0)
+    (property "Reference" "J**1" (at 161.29 156.21 0)
+      (effects (font (size 2.54 2.54)))
+    )
+    (property "Value" "SolderWire-0.25sqmm_1x20_P4.2mm_D0.65mm_OD1.7mm" (at 165.1 125.73 90)
+      (effects (font (size 1.27 1.27)))
+    )
+    (property "Footprint" "PG:b_pill_takeoffPads_1-20" (at 167.64 130.81 90) (show_name)
+      (effects (font (size 1.27 1.27)))
+    )
+    (property "Datasheet" "" (at 147.32 128.27 0)
       (effects (font (size 1.27 1.27)) hide)
     )
@@
       (project "ads1115with16JTS"
         (path "/0c2d0c14-8850-4a30-bb78-b2f40cb442ba"
-          (reference "pads2") (unit 1)
+          (reference "J**1") (unit 1)
         )
       )
@@
     )
   )
-  (symbol (lib_id "PG:b_pill_21-40") (at 167.64 128.27 0) (unit 1)
+  (symbol (lib_id "PG:b_pill_takeoff_21-40") (at 167.64 128.27 0) (unit 1)
     (in_bom yes) (on_board yes) (dnp no)
-    (property "Reference" "pads3" (at 179.07 156.21 0)
+    (property "Reference" "J**2" (at 182.88 156.21 0)
       (effects (font (size 2.54 2.54)))
     )
-    (property "Value" "SolderWire-0.25sqmm_1x20_P4.2mm_D0.65mm_OD1.7mm\n" (at 175.26 124.46 90)
-      (effects (font (size 1.27 1.27)))
-    )
-    (property "Footprint" "PG:b_pill_takeoffPads_21-40" (at 172.72 129.54 90) (show_name)
+    (property "Value" "SolderWire-0.25sqmm_1x20_P4.2mm_D0.65mm_OD1.7mm" (at 177.8 128.27 90)
+      (effects (font (size 1.27 1.27)))
+    )
+    (property "Footprint" "PG:b_pill_takeoffPads_21-40" (at 175.26 130.81 90) (show_name)
       (effects (font (size 1.27 1.27)))
     )
@@
       (project "ads1115with16JTS"
         (path "/0c2d0c14-8850-4a30-bb78-b2f40cb442ba"
-          (reference "pads3") (unit 1)
-        )
-      )
+          (reference "J**2") (unit 1)
+        )
+      )

Commit message: v0.0.14 snapshot.
Parts:
- added H1, H2: MountingHole, MountingHole:MountingHole_2.2mm_M2_ISO7380_Pad, symbol Mechanical:MountingHole
Connections:
- net GND: now also J**1.19, J18.19 (G)
Changed lines of the file:
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@@
   (junction (at 140.97 67.31) (diameter 0) (color 0 0 0 0)
   )
+  (junction (at 168.91 148.59) (diameter 0) (color 0 0 0 0)
+  )
   (junction (at 125.73 171.45) (diameter 0) (color 0 0 0 0)
   )
@@
   )
   (junction (at 190.5 55.88) (diameter 0) (color 0 0 0 0)
+  )
+  (junction (at 162.56 148.59) (diameter 0) (color 0 0 0 0)
   )
   (junction (at 125.73 85.09) (diameter 0) (color 0 0 0 0)
@@
     (stroke (width 0) (type default))
   )
+  (wire (pts (xy 168.91 148.59) (xy 168.91 149.86))
+    (stroke (width 0) (type default))
+  )
   (wire (pts (xy 157.48 128.27) (xy 162.56 128.27))
     (stroke (width 0) (type default))
@@
   )
   (wire (pts (xy 143.51 104.14) (xy 143.51 161.29))
+    (stroke (width 0) (type default))
+  )
+  (wire (pts (xy 162.56 148.59) (xy 168.91 148.59))
     (stroke (width 0) (type default))
   )
@@
   (symbol (lib_id "PG:b_pill_21-40") (at 207.01 128.27 0) (mirror y) (unit 1)
     (in_bom yes) (on_board yes) (dnp no)
-    (property "Reference" "J19" (at 195.58 156.21 0)
+    (property "Reference" "J19" (at 197.01 155.27 0)
       (effects (font (size 2.54 2.54)))
     )
-    (property "Value" "PinSocket_1x20_P2.54mm_Vertical" (at 199.39 132.08 90)
-      (effects (font (size 1.27 1.27)))
-    )
-    (property "Footprint" "PG:b_pill_socket_21-40" (at 201.93 132.08 90) (show_name)
+    (property "Value" "PinSocket_1x20_P2.54mm_Vertical" (at 200.66 128.27 90)
+      (effects (font (size 1.27 1.27)))
+    )
+    (property "Footprint" "PG:b_pill_socket_21-40" (at 203.2 128.27 90) (show_name)
       (effects (font (size 1.27 1.27)))
     )
@@
   (symbol (lib_id "PG:b_pill_1-20") (at 157.48 128.27 0) (unit 1)
     (in_bom yes) (on_board yes) (dnp no)
-    (property "Reference" "J18" (at 151.13 156.21 0)
+    (property "Reference" "J18" (at 149.86 154.94 0)
       (effects (font (size 2.54 2.54)) (justify left))
     )
-    (property "Value" "PinSocket_1x20_P2.54mm_Vertical" (at 149.86 140.97 90)
-      (effects (font (size 1.27 1.27)) (justify left))
-    )
-    (property "Footprint" "PG:b_pill_socket_1-20" (at 147.32 139.7 90) (show_name)
+    (property "Value" "PinSocket_1x20_P2.54mm_Vertical" (at 148.59 144.78 90)
+      (effects (font (size 1.27 1.27)) (justify left))
+    )
+    (property "Footprint" "PG:b_pill_socket_1-20" (at 146.05 144.78 90) (show_name)
       (effects (font (size 1.27 1.27)) (justify left))
     )
@@
     )
   )
+  (symbol (lib_id "power:PWR_FLAG") (at 168.91 148.59 0) (unit 1)
+    (in_bom yes) (on_board yes) (dnp no) (fields_autoplaced)
+    (property "Reference" "#FLG03" (at 168.91 146.685 0)
+      (effects (font (size 1.27 1.27)) hide)
+    )
+    (property "Value" "PWR_FLAG" (at 168.91 143.51 0)
+      (effects (font (size 1.27 1.27)))
+    )
+    (property "Footprint" "" (at 168.91 148.59 0)
+      (effects (font (size 1.27 1.27)) hide)
+    )
+    (property "Datasheet" "~" (at 168.91 148.59 0)
+      (effects (font (size 1.27 1.27)) hide)
+    )
+    (pin "1")
+    (instances
+      (project "ads1115with16JTS"
+        (path "/0c2d0c14-8850-4a30-bb78-b2f40cb442ba"
+          (reference "#FLG03") (unit 1)
+        )
+      )
+    )
+  )
   (symbol (lib_id "Connector:Conn_01x02_Pin") (at 43.18 184.15 0) (unit 1)
     (in_bom yes) (on_board yes) (dnp no)
@@
   (symbol (lib_id "PG:b_pill_takeoff_1-20") (at 160.02 128.27 0) (mirror y) (unit 1)
     (in_bom yes) (on_board yes) (dnp no)
-    (property "Reference" "J**1" (at 161.29 156.21 0)
+    (property "Reference" "J**1" (at 166.37 157.48 0)
       (effects (font (size 2.54 2.54)))
     )
@@
     )
   )
+  (symbol (lib_id "Mechanical:MountingHole") (at 170.18 227.33 0) (unit 1)
+    (in_bom yes) (on_board yes) (dnp no) (fields_autoplaced)
+    (property "Reference" "H1" (at 172.72 226.06 0)
+      (effects (font (size 1.27 1.27)) (justify left))
+    )
+    (property "Value" "MountingHole" (at 172.72 228.6 0)
+      (effects (font (size 1.27 1.27)) (justify left))
+    )
+    (property "Footprint" "MountingHole:MountingHole_2.2mm_M2_ISO7380_Pad" (at 170.18 227.33 0)
+      (effects (font (size 1.27 1.27)) hide)
+    )
+    (property "Datasheet" "~" (at 170.18 227.33 0)
+      (effects (font (size 1.27 1.27)) hide)
+    )
+    (instances
+      (project "ads1115with16JTS"
+        (path "/0c2d0c14-8850-4a30-bb78-b2f40cb442ba"
+          (reference "H1") (unit 1)
+        )
+      )
+    )
+  )
   (symbol (lib_id "power:GND") (at 48.26 41.91 0) (unit 1)
     (in_bom yes) (on_board yes) (dnp no) (fields_autoplaced)
@@
     )
   )
+  (symbol (lib_id "Mechanical:MountingHole") (at 152.4 20.32 0) (unit 1)
+    (in_bom yes) (on_board yes) (dnp no) (fields_autoplaced)
+    (property "Reference" "H2" (at 154.94 19.05 0)
+      (effects (font (size 1.27 1.27)) (justify left))
+    )
+    (property "Value" "MountingHole" (at 154.94 21.59 0)
+      (effects (font (size 1.27 1.27)) (justify left))
+    )
+    (property "Footprint" "MountingHole:MountingHole_2.2mm_M2_ISO7380_Pad" (at 152.4 20.32 0)
+      (effects (font (size 1.27 1.27)) hide)
+    )
+    (property "Datasheet" "~" (at 152.4 20.32 0)
+      (effects (font (size 1.27 1.27)) hide)
+    )
+    (instances
+      (project "ads1115with16JTS"
+        (path "/0c2d0c14-8850-4a30-bb78-b2f40cb442ba"
+          (reference "H2") (unit 1)
+        )
+      )
+    )
+  )
   (symbol (lib_id "power:+3V3") (at 81.28 165.1 0) (unit 1)
     (in_bom yes) (on_board yes) (dnp no) (fields_autoplaced)
@@
         )
       )
+    )
+  )
+  (symbol (lib_id "power:GND") (at 168.91 149.86 0) (unit 1)
+    (in_bom yes) (on_board yes) (dnp no) (fields_autoplaced)
+    (property "Reference" "#PWR049" (at 168.91 156.21 0)
+      (effects (font (size 1.27 1.27)) hide)
+    )
+    (property "Value" "GND" (at 168.91 154.94 0)
+      (effects (font (size 1.27 1.27)))
+    )
+    (property "Footprint" "" (at 168.91 149.86 0)
+      (effects (font (size 1.27 1.27)) hide)
+    )
+    (property "Datasheet" "" (at 168.91 149.86 0)
+      (effects (font (size 1.27 1.27)) hide)
+    )
+    (pin "1")
+    (instances
+      (project "ads1115with16JTS"
+        (path "/0c2d0c14-8850-4a30-bb78-b2f40cb442ba"
+          (reference "#PWR049") (unit 1)
+        )
+      )
