File: SensorProject_t16-pcb.kicad_sch (KiCad schematic)
At the start: 50 parts, among them J1 Conn_01x02_Pin, J10 Conn_01x02_Pin, J11 Conn_01x02_Pin, J12 Conn_01x02_Pin, J13 Conn_01x02_Pin, J14 Conn_01x02_Pin, J15 Conn_01x02_Pin, J16 Conn_01x02_Pin, J2 Conn_01x02_Pin, J3 Conn_01x02_Pin, J4 Conn_01x02_Pin, J5 Conn_01x02_Pin, J6 Conn_01x02_Pin, J7 Conn_01x02_Pin, J8 Conn_01x02_Pin, J9 Conn_01x02_Pin, U1 ADS1115IDGS, U2 ADS1115IDGS, U3 ADS1115IDGS, U4 ADS1115IDGS

Commit message: improved schematic sheet titles.
Other:
- title: ADCs for 10K thermistors -> ADC and 16 10K thermistors - MCU + LoRa
Changed lines of the file:
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@@
 	(paper "A" portrait)
 	(title_block
-		(title "ADCs for 10K thermistors")
-		(date "2025-01-07")
-		(rev "v0.1.1")
+		(title "ADC and 16 10K thermistors - MCU + LoRa")
+		(date "2025-09-15")
+		(rev "v0.2.2")
 	)
 	(junction

Commit message: added caps to radio_gnd.
Parts:
- C1, C2, C3, C4: value 0.1µF -> 100nF; Manufacturer (none) -> Yageo; MfgPart (none) -> CC0402KRX7R7BB104
Changed lines of the file:
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@@
 			)
 		)
-		(property "Value" "0.1µF"
+		(property "Value" "100nF"
 			(at 120.65 88.9 90)
 			(show_name no)
@@
 			)
 		)
-		(property "Manufacturer" ""
+		(property "Manufacturer" "Yageo"
 			(at 120.65 85.09 90)
 			(hide yes)
@@
 			)
 		)
-		(property "MfgPart" ""
+		(property "MfgPart" "CC0402KRX7R7BB104"
 			(at 120.65 85.09 90)
 			(hide yes)
@@
 			)
 		)
-		(property "Value" "0.1µF"
+		(property "Value" "100nF"
 			(at 120.65 27.94 90)
 			(show_name no)
@@
 			)
 		)
-		(property "Manufacturer" ""
+		(property "Manufacturer" "Yageo"
 			(at 120.65 24.13 90)
 			(hide yes)
@@
 			)
 		)
-		(property "MfgPart" ""
+		(property "MfgPart" "CC0402KRX7R7BB104"
 			(at 120.65 24.13 90)
 			(hide yes)
@@
 			)
 		)
-		(property "Value" "0.1µF"
+		(property "Value" "100nF"
 			(at 123.19 200.66 90)
 			(show_name no)
@@
 			)
 		)
-		(property "Manufacturer" ""
+		(property "Manufacturer" "Yageo"
 			(at 123.19 196.85 90)
 			(hide yes)
@@
 			)
 		)
-		(property "MfgPart" ""
+		(property "MfgPart" "CC0402KRX7R7BB104"
 			(at 123.19 196.85 90)
 			(hide yes)
@@
 			)
 		)
-		(property "Value" "0.1µF"
+		(property "Value" "100nF"
 			(at 120.65 146.05 90)
 			(show_name no)
@@
 			)
 		)
-		(property "Manufacturer" ""
+		(property "Manufacturer" "Yageo"
 			(at 120.65 142.24 90)
 			(hide yes)
@@
 			)
 		)
-		(property "MfgPart" ""
+		(property "MfgPart" "CC0402KRX7R7BB104"
 			(at 120.65 142.24 90)
 			(hide yes)

Commit message: Cleaned up v0.3.0 2026-04. LSE and HSE populated.
Parts:
- C1, C2, C3, C4: Manufacturer Yageo -> (none); MfgPart CC0402KRX7R7BB104 -> (none)
Changed lines of the file:
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@@
 			)
 		)
-		(property "Manufacturer" "Yageo"
+		(property "Manufacturer" ""
 			(at 120.65 85.09 90)
 			(hide yes)
@@
 			)
 		)
-		(property "MfgPart" "CC0402KRX7R7BB104"
+		(property "MfgPart" ""
 			(at 120.65 85.09 90)
 			(hide yes)
@@
 			)
 		)
-		(property "Manufacturer" "Yageo"
+		(property "Manufacturer" ""
 			(at 120.65 24.13 90)
 			(hide yes)
@@
 			)
 		)
-		(property "MfgPart" "CC0402KRX7R7BB104"
+		(property "MfgPart" ""
 			(at 120.65 24.13 90)
 			(hide yes)
@@
 			)
 		)
-		(property "Manufacturer" "Yageo"
+		(property "Manufacturer" ""
 			(at 123.19 196.85 90)
 			(hide yes)
@@
 			)
 		)
-		(property "MfgPart" "CC0402KRX7R7BB104"
+		(property "MfgPart" ""
 			(at 123.19 196.85 90)
 			(hide yes)
@@
 			)
 		)
-		(property "Manufacturer" "Yageo"
+		(property "Manufacturer" ""
 			(at 120.65 142.24 90)
 			(hide yes)
@@
 			)
 		)
-		(property "MfgPart" "CC0402KRX7R7BB104"
+		(property "MfgPart" ""
 			(at 120.65 142.24 90)
 			(hide yes)

Commit message: added QR and ID blocks on silkscreen. Marked HSE and LSE as DNP. Revised version number to 0.3.1.
Other:
- title: ADC and 16 10K thermistors - MCU + LoRa -> stm32f411, RFM95W
Changed lines of the file:
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@@
 	(paper "A" portrait)
 	(title_block
-		(title "ADC and 16 10K thermistors - MCU + LoRa")
-		(date "2025-09-15")
-		(rev "v0.2.2")
+		(title "stm32f411, RFM95W")
+		(date "2026-04-12")
+		(rev "v0.3.1")
 	)
 	(junction
